Commit message: Added support for Baxter Robot

File: urdf/ur5_robot.urdf (robot description, URDF)
Before this commit: robot ur5, 9 links, 8 joints
Links:
- link base_link: geometry visual mesh filename=package://ur_description/meshes/ur5/visual/base.dae
- link forearm_link: geometry visual mesh filename=package://ur_description/meshes/ur5/visual/forearm.dae
- link shoulder_link: geometry visual mesh filename=package://ur_description/meshes/ur5/visual/shoulder.dae
- link upper_arm_link: geometry visual mesh filename=package://ur_description/meshes/ur5/visual/upperarm.dae
- link wrist_1_link: geometry visual mesh filename=package://ur_description/meshes/ur5/visual/wrist1.dae
- link wrist_2_link: geometry visual mesh filename=package://ur_description/meshes/ur5/visual/wrist2.dae
- link wrist_3_link: geometry visual mesh filename=package://ur_description/meshes/ur5/visual/wrist3.dae
